File: xx_backplane_shield_xi.brd (EAGLE design)
At the start: 80 x 82.5 mm, 27 parts

Commit message: Added connector and mosfet for OBS
Parts:
- added LED9: (no value), led:SML0603
- added POWER2: T2I5P, T2I5P:T2I5P
- added R6: 330, resistor:R0603
- added U1: FQB27P06, CamSensComponents:TO263-3
Connections:
- new net E_MAG_1: POWER2.P$5, POWER2.P$6, R6.2, U1.TAB
- new net E_MAG_1_ON: PCB1.P$35, U1.1
- new net N$51: LED9.A, R6.1
- net +5V: now also U1.3
- net GND: now also LED9.C, POWER2.P$2, POWER2.P$3
Routing:
- net E_MAG_1: track 0.00 -> 26.6 mm
- net E_MAG_1_ON: track 0.00 -> 11.1 mm
- net +5V: track 265.5 -> 269.0 mm, vias 6 -> 7
- net N$51: track 0.00 -> 1.19 mm
Other:
- board text added: "+5V"
- board text added: "GND"
- board text added: "OBS"
- board text added: "Power"
Changed lines of the file:
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@@
 Luke McBee
 Ryan McBee</text>
+<text x="20.066" y="54.102" size="1.778" layer="22" rot="MR0">OBS</text>
+<text x="20.574" y="69.342" size="1.778" layer="22" rot="MR0">Power</text>
+<text x="-0.762" y="66.04" size="1.778" layer="22" rot="MR0">Power</text>
+<text x="-2.54" y="41.148" size="1.778" layer="21">+5V</text>
+<text x="59.436" y="40.894" size="1.778" layer="21">GND</text>
 </plain>
 <attributes>
@@
 <element name="C5" library="SparkFun-Passives" package="0603-CAP" value="0.1u" x="31.75" y="21.59" rot="R270"/>
 <element name="C6" library="SparkFun-Passives" package="0603-CAP" value="0.1u" x="41.148" y="22.606" rot="R270"/>
+<element name="U1" library="CamSensComponents" package="TO263-3" value="FQB27P06" x="46.99" y="55.118" rot="MR180"/>
+<element name="R6" library="resistor" package="R0603" value="330" x="39.624" y="50.292" rot="MR180"/>
+<element name="LED9" library="led" package="SML0603" value="" x="36.83" y="50.292" rot="MR180"/>
+<element name="POWER2" library="T2I5P" package="T2I5P" value="T2I5P" x="21.336" y="58.166" rot="R180"/>
 </elements>
 <signals>
@@
 <via x="9.3218" y="54.7116" extent="1-16" drill="0.45"/>
 <via x="9.017" y="50.9778" extent="1-16" drill="0.45"/>
-<via x="47.4472" y="55.7784" extent="1-16" drill="0.45"/>
 <via x="12.4968" y="49.784" extent="1-16" drill="0.45"/>
 <via x="16.3068" y="39.9288" extent="1-16" drill="0.45"/>
@@
 <via x="29.7688" y="51.1556" extent="1-16" drill="0.45"/>
 <via x="39.0398" y="55.9816" extent="1-16" drill="0.45"/>
-<via x="39.0398" y="50.4444" extent="1-16" drill="0.45"/>
 <via x="38.1" y="44.6532" extent="1-16" drill="0.45"/>
 <via x="5.1308" y="36.6522" extent="1-16" drill="0.45"/>
@@
 <contactref element="C6" pad="1"/>
 <via x="32.512" y="59.944" extent="1-16" drill="0.35"/>
+<contactref element="LED9" pad="C"/>
+<contactref element="POWER2" pad="P$2"/>
+<contactref element="POWER2" pad="P$3"/>
 </signal>
 <signal name="+5V">
@@
 <wire x1="28.2702" y1="20.6756" x2="28.2702" y2="17.7038" width="0.8128" layer="16"/>
 <wire x1="28.2702" y1="17.7038" x2="28.448" y2="17.526" width="0.8128" layer="16"/>
+<contactref element="U1" pad="3"/>
+<wire x1="49.53" y1="60.198" x2="51.562" y2="60.198" width="0.4064" layer="16"/>
+<via x="51.562" y="60.198" extent="1-16" drill="0.35"/>
+<wire x1="51.562" y1="60.198" x2="51.562" y2="60.5028" width="0.4064" layer="1"/>
+<wire x1="51.562" y1="60.5028" x2="52.324" y2="61.2648" width="0.4064" layer="1"/>
 </signal>
 <signal name="3.3V">
@@
 </polygon>
 </signal>
+<signal name="N$51">
+<contactref element="R6" pad="1"/>
+<contactref element="LED9" pad="A"/>
+<wire x1="38.774" y1="50.292" x2="37.58" y2="50.292" width="0.4064" layer="16"/>
+</signal>
+<signal name="E_MAG_1">
+<contactref element="U1" pad="TAB"/>
+<contactref element="R6" pad="2"/>
+<contactref element="POWER2" pad="P$5"/>
+<contactref element="POWER2" pad="P$6"/>
+<wire x1="40.474" y1="50.292" x2="41.2487" y2="49.5173" width="0.4064" layer="16"/>
+<wire x1="41.2487" y1="49.5173" x2="46.99" y2="49.5173" width="0.4064" layer="16"/>
+<wire x1="40.474" y1="50.292" x2="38.188" y2="52.578" width="0.4064" layer="16"/>
+<wire x1="38.188" y1="52.578" x2="26.67" y2="52.578" width="0.4064" layer="16"/>
+<wire x1="26.67" y1="52.578" x2="25.036" y2="54.212" width="0.4064" layer="16"/>
+<wire x1="25.036" y1="54.212" x2="25.036" y2="54.864" width="0.4064" layer="16"/>
+<wire x1="25.036" y1="54.864" x2="25.036" y2="54.866" width="0.4064" layer="16"/>
+<wire x1="27.036" y1="54.866" x2="27.034" y2="54.864" width="0.4064" layer="16"/>
+<wire x1="27.034" y1="54.864" x2="25.036" y2="54.864" width="0.4064" layer="16"/>
+</signal>
+<signal name="E_MAG_1_ON">
+<contactref element="U1" pad="1"/>
+<wire x1="44.45" y1="60.198" x2="47.752" y2="63.5" width="0.4064" layer="16"/>
+<contactref element="PCB1" pad="P$35"/>
+<wire x1="52.7304" y1="63.5" x2="53.7718" y2="62.4586" width="0.4064" layer="16"/>
+<wire x1="47.752" y1="63.5" x2="52.7304" y2="63.5" width="0.4064" layer="16"/>
+</signal>
 </signals>
+<errors>
+</errors>
 </board>
 </drawing>
