File: xx_backplane_shield_xi.brd (EAGLE design)
At the start: 80 x 82.5 mm, 31 parts, among them U1 FQB27P06

Commit message: Added servo motor connection
Parts:
- added SV1: (no value), con-lstb:MA03-1
Connections:
- new net SERVO_PWM: PCB1.P$33, SV1.1
- net +5V: now also SV1.2
- net GND: now also SV1.3
Routing:
- net SERVO_PWM: track 0.00 -> 20.9 mm, vias 0 -> 2
- net +5V: track 269.0 -> 280.4 mm
Other:
- board text added: "+5v"
- board text added: "gnd"
- board text added: "pwm"
Changed lines of the file:
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@@
 <?xml version="1.0" encoding="utf-8"?>
 <!DOCTYPE eagle SYSTEM "eagle.dtd">
-<eagle version="8.4.1">
+<eagle version="8.5.2">
 <drawing>
 <settings>
@@
 <text x="-2.54" y="41.148" size="1.778" layer="21">+5V</text>
 <text x="59.436" y="40.894" size="1.778" layer="21">GND</text>
+<text x="48.768" y="67.31" size="1.016" layer="21">pwm</text>
+<text x="49.022" y="72.644" size="1.016" layer="21">gnd</text>
+<text x="49.022" y="69.85" size="1.016" layer="21">+5v</text>
 </plain>
 <attributes>
@@
 <param name="checkRestrict" value="0"/>
 <param name="checkStop" value="0"/>
+<param name="checkValues" value="0"/>
 <param name="useDiameter" value="13"/>
 <param name="maxErrors" value="50"/>
@@
 <element name="LED9" library="led" package="SML0603" value="" x="36.83" y="50.292" rot="MR180"/>
 <element name="POWER2" library="T2I5P" package="T2I5P" value="T2I5P" x="21.336" y="58.166" rot="R180"/>
+<element name="SV1" library="con-lstb" library_urn="urn:adsk.eagle:library:162" package="MA03-1" package3d_urn="urn:adsk.eagle:package:8339/1" value="" x="46.736" y="70.104" rot="R90">
+<attribute name="MF" value="" x="46.736" y="70.104" size="1.778" layer="27" rot="R90" display="off"/>
+<attribute name="MPN" value="" x="46.736" y="70.104" size="1.778" layer="27" rot="R90" display="off"/>
+<attribute name="OC_FARNELL" value="unknown" x="46.736" y="70.104" size="1.778" layer="27" rot="R90" display="off"/>
+<attribute name="OC_NEWARK" value="unknown" x="46.736" y="70.104" size="1.778" layer="27" rot="R90" display="off"/>
+</element>
 </elements>
 <signals>
@@
 <via x="36.7792" y="66.0908" extent="1-16" drill="0.45"/>
 <via x="36.6268" y="70.9676" extent="1-16" drill="0.45"/>
-<via x="43.9166" y="71.0946" extent="1-16" drill="0.45"/>
+<via x="43.6626" y="73.6346" extent="1-16" drill="0.45"/>
 <via x="44.2722" y="65.6336" extent="1-16" drill="0.45"/>
-<via x="48.1076" y="71.7804" extent="1-16" drill="0.45"/>
+<via x="41.7576" y="72.5424" extent="1-16" drill="0.45"/>
 <via x="50.0634" y="64.8716" extent="1-16" drill="0.45"/>
 <via x="59.9948" y="68.4022" extent="1-16" drill="0.45"/>
@@
 <contactref element="POWER2" pad="P$3"/>
 <via x="1.016" y="72.136" extent="1-16" drill="0.35"/>
+<contactref element="SV1" pad="3"/>
 </signal>
 <signal name="+5V">
@@
 <wire x1="-6.2484" y1="71.247" x2="-6.2484" y2="66.4316" width="0.4064" layer="1"/>
 <wire x1="-6.26" y1="66.42" x2="-6.2484" y2="66.4316" width="0.4064" layer="1"/>
-<wire x1="51.5366" y1="62.0522" x2="34.8234" y2="62.0522" width="0.8128" layer="1"/>
 <wire x1="51.5366" y1="62.0522" x2="52.324" y2="61.2648" width="0.8128" layer="1"/>
 <wire x1="52.324" y1="61.2648" x2="60.833" y2="61.2902" width="0.4064" layer="1"/>
@@
 <contactref element="POWER1" pad="P$6"/>
 <wire x1="27.0868" y1="69.7888" x2="27.0868" y2="69.9282" width="0.8128" layer="1"/>
-<wire x1="34.8234" y1="62.0522" x2="27.0868" y2="69.7888" width="0.8128" layer="1"/>
 <wire x1="13.335" y1="72.0344" x2="22.9806" y2="72.0344" width="1.524" layer="16"/>
 <wire x1="22.9806" y1="72.0344" x2="25.0868" y2="69.9282" width="1.524" layer="16"/>
@@
 <wire x1="51.562" y1="60.198" x2="51.562" y2="60.5028" width="0.4064" layer="1"/>
 <wire x1="51.562" y1="60.5028" x2="52.324" y2="61.2648" width="0.4064" layer="1"/>
+<contactref element="SV1" pad="2"/>
+<wire x1="46.736" y1="70.104" x2="44.196" y2="70.104" width="0.8128" layer="1"/>
+<wire x1="44.196" y1="70.104" x2="41.656" y2="67.564" width="0.8128" layer="1"/>
+<wire x1="41.656" y1="67.564" x2="41.656" y2="63.5" width="0.8128" layer="1"/>
+<wire x1="41.656" y1="63.5" x2="40.132" y2="61.976" width="0.8128" layer="1"/>
+<wire x1="40.132" y1="61.976" x2="34.8996" y2="61.976" width="0.8128" layer="1"/>
+<wire x1="34.8996" y1="61.976" x2="27.0868" y2="69.7888" width="0.8128" layer="1"/>
+<wire x1="41.656" y1="63.5" x2="43.1038" y2="62.0522" width="0.8128" layer="1"/>
+<wire x1="43.1038" y1="62.0522" x2="51.5366" y2="62.0522" width="0.8128" layer="1"/>
 </signal>
 <signal name="3.3V">
@@
 <wire x1="47.752" y1="63.5" x2="52.7304" y2="63.5" width="0.4064" layer="16"/>
 </signal>
+<signal name="SERVO_PWM">
+<contactref element="PCB1" pad="P$33"/>
+<contactref element="SV1" pad="1"/>
+<wire x1="46.736" y1="67.564" x2="46.736" y2="65.532" width="0.3048" layer="1"/>
+<wire x1="46.736" y1="65.532" x2="44.704" y2="63.5" width="0.3048" layer="1"/>
+<via x="44.704" y="63.5" extent="1-16" drill="0.35"/>
+<via x="42.926" y="60.452" extent="1-16" drill="0.35"/>
+<wire x1="42.926" y1="60.452" x2="43.942" y2="59.436" width="0.3048" layer="1"/>
+<wire x1="53.2892" y1="59.436" x2="53.7718" y2="59.9186" width="0.3048" layer="1"/>
+<wire x1="43.942" y1="59.436" x2="53.2892" y2="59.436" width="0.3048" layer="1"/>
+<wire x1="42.926" y1="62.992" x2="43.434" y2="63.5" width="0.3048" layer="16"/>
+<wire x1="43.434" y1="63.5" x2="44.704" y2="63.5" width="0.3048" layer="16"/>
+<wire x1="42.926" y1="60.452" x2="42.926" y2="62.992" width="0.3048" layer="16"/>
+</signal>
 </signals>
