File: xx_backplane_shield_xi.sch (EAGLE design)
At the start: 25 parts

Commit message: Updated traces and changed connector for main camera
Parts:
- removed USB_CAM_POW: (no value), pinhead:PINHD-1X3
- added C5, C6: 0.1u, SparkFun-Passives:CAP0603-CAP
- added POWER1: USB_CAM_POW, T2I5P:T2I5P
Connections:
- net +5V: now also C5.2, POWER1.4, POWER1.5; no longer USB_CAM_POW.1
- net 3.3V: now also C6.2
- net GND: now also C5.1, C6.1, POWER1.1, POWER1.2; no longer USB_CAM_POW.3
Changed lines of the file:
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@@
 <?xml version="1.0" encoding="utf-8"?>
 <!DOCTYPE eagle SYSTEM "eagle.dtd">
-<eagle version="8.3.2">
+<eagle version="8.4.3">
 <drawing>
 <settings>
@@
 <part name="R5" library="resistor" library_urn="urn:adsk.eagle:library:348" deviceset="R-US_" device="R0603" package3d_urn="urn:adsk.eagle:package:26057/1" value="0 ohms"/>
 <part name="PS2" library="con-hirose-df13" deviceset="DF13-4P-1.25" device="DSA"/>
-<part name="USB_CAM_POW" library="pinhead" library_urn="urn:adsk.eagle:library:325" deviceset="PINHD-1X3" device="" package3d_urn="urn:adsk.eagle:package:22458/2"/>
 <part name="C2" library="SparkFun-Passives" deviceset="CAP" device="0603-CAP" value="0.1u"/>
 <part name="C4" library="SparkFun-Passives" deviceset="CAP" device="0603-CAP" value="0.1u"/>
 <part name="GND7" library="SparkFun-Aesthetics" deviceset="GND" device=""/>
 <part name="GND14" library="SparkFun-Aesthetics" deviceset="GND" device=""/>
+<part name="POWER1" library="T2I5P" deviceset="T2I5P" device="" value="USB_CAM_POW"/>
+<part name="C5" library="SparkFun-Passives" deviceset="CAP" device="0603-CAP" value="0.1u"/>
+<part name="C6" library="SparkFun-Passives" deviceset="CAP" device="0603-CAP" value="0.1u"/>
 </parts>
 <sheets>
@@
 <instance part="FRAME2" gate="G$1" x="-276.86" y="0"/>
 <instance part="FRAME2" gate="G$2" x="-104.14" y="0"/>
-<instance part="FRAME3" gate="G$1" x="2.54" y="2.54"/>
+<instance part="FRAME3" gate="G$1" x="2.54" y="0"/>
 <instance part="FRAME3" gate="G$2" x="175.26" y="0"/>
 <instance part="PCB1" gate="G$1" x="-137.16" y="33.02" rot="R90"/>
@@
 <instance part="GND11" gate="1" x="-248.92" y="86.36"/>
 <instance part="GND12" gate="1" x="-246.38" y="111.76"/>
-<instance part="GND2" gate="1" x="132.08" y="170.18" smashed="yes">
-<attribute name="VALUE" x="129.54" y="167.64" size="1.778" layer="96"/>
+<instance part="GND2" gate="1" x="132.08" y="162.56" smashed="yes">
+<attribute name="VALUE" x="129.54" y="160.02" size="1.778" layer="96"/>
 </instance>
 <instance part="LED5" gate="G$1" x="-50.8" y="177.8"/>
@@
 <attribute name="NAME" x="-52.705" y="134.62" size="1.778" layer="95"/>
 </instance>
-<instance part="USB_CAM_POW" gate="A" x="-48.26" y="58.42"/>
 <instance part="C2" gate="G$1" x="96.52" y="121.92"/>
 <instance part="C4" gate="G$1" x="157.48" y="121.92"/>
 <instance part="GND7" gate="1" x="96.52" y="114.3"/>
 <instance part="GND14" gate="1" x="157.48" y="114.3"/>
+<instance part="POWER1" gate="&gt;NAME" x="-22.86" y="81.28" rot="R270"/>
+<instance part="C5" gate="G$1" x="114.3" y="177.8" rot="R180"/>
+<instance part="C6" gate="G$1" x="147.32" y="177.8" rot="MR180"/>
 </instances>
 <busses>
@@
 <segment>
 <pinref part="U$5" gate="G$1" pin="GND"/>
-<wire x1="132.08" y1="172.72" x2="132.08" y2="175.26" width="0.1524" layer="91"/>
+<wire x1="132.08" y1="165.1" x2="132.08" y2="170.18" width="0.1524" layer="91"/>
 <pinref part="GND2" gate="1" pin="GND"/>
+<pinref part="C5" gate="G$1" pin="1"/>
+<wire x1="132.08" y1="170.18" x2="132.08" y2="175.26" width="0.1524" layer="91"/>
+<wire x1="114.3" y1="172.72" x2="114.3" y2="170.18" width="0.1524" layer="91"/>
+<wire x1="114.3" y1="170.18" x2="132.08" y2="170.18" width="0.1524" layer="91"/>
+<junction x="132.08" y="170.18"/>
+<pinref part="C6" gate="G$1" pin="1"/>
+<wire x1="147.32" y1="172.72" x2="147.32" y2="170.18" width="0.1524" layer="91"/>
+<wire x1="147.32" y1="170.18" x2="132.08" y2="170.18" width="0.1524" layer="91"/>
 </segment>
 <segment>
@@
 </segment>
 <segment>
-<pinref part="USB_CAM_POW" gate="A" pin="3"/>
-<wire x1="-50.8" y1="55.88" x2="-66.04" y2="55.88" width="0.1524" layer="91"/>
-<label x="-66.04" y="55.88" size="1.778" layer="95"/>
-</segment>
-<segment>
 <pinref part="C2" gate="G$1" pin="2"/>
 <pinref part="GND7" gate="1" pin="GND"/>
@@
 <pinref part="GND14" gate="1" pin="GND"/>
 <wire x1="157.48" y1="119.38" x2="157.48" y2="116.84" width="0.1524" layer="91"/>
+</segment>
+<segment>
+<pinref part="POWER1" gate="&gt;NAME" pin="1"/>
+<wire x1="-27.94" y1="86.36" x2="-35.56" y2="86.36" width="0.1524" layer="91"/>
+<label x="-35.56" y="86.36" size="1.778" layer="95"/>
+</segment>
+<segment>
+<pinref part="POWER1" gate="&gt;NAME" pin="2"/>
+<wire x1="-27.94" y1="83.82" x2="-35.56" y2="83.82" width="0.1524" layer="91"/>
+<label x="-35.56" y="83.82" size="1.778" layer="95"/>
 </segment>
 </net>
@@
 <pinref part="U$5" gate="G$1" pin="VIN"/>
 <wire x1="121.92" y1="182.88" x2="114.3" y2="182.88" width="0.1524" layer="91"/>
+<pinref part="C5" gate="G$1" pin="2"/>
+<wire x1="114.3" y1="180.34" x2="114.3" y2="182.88" width="0.1524" layer="91"/>
+<junction x="114.3" y="182.88"/>
 </segment>
 <segment>
@@
 </segment>
 <segment>
-<pinref part="USB_CAM_POW" gate="A" pin="1"/>
-<wire x1="-50.8" y1="60.96" x2="-66.04" y2="60.96" width="0.1524" layer="91"/>
-<label x="-66.04" y="60.96" size="1.778" layer="95"/>
+<pinref part="POWER1" gate="&gt;NAME" pin="4"/>
+<wire x1="-27.94" y1="78.74" x2="-35.56" y2="78.74" width="0.1524" layer="91"/>
+<label x="-35.56" y="78.74" size="1.778" layer="95"/>
+</segment>
+<segment>
+<pinref part="POWER1" gate="&gt;NAME" pin="5"/>
+<wire x1="-27.94" y1="76.2" x2="-35.56" y2="76.2" width="0.1524" layer="91"/>
+<label x="-35.56" y="76.2" size="1.778" layer="95"/>
 </segment>
 </net>
@@
 <wire x1="144.78" y1="182.88" x2="147.32" y2="182.88" width="0.1524" layer="91"/>
 <wire x1="147.32" y1="182.88" x2="147.32" y2="187.96" width="0.1524" layer="91"/>
-</segment>
-<segment>
+<pinref part="C6" gate="G$1" pin="2"/>
+<wire x1="147.32" y1="180.34" x2="147.32" y2="182.88" width="0.1524" layer="91"/>
+<junction x="147.32" y="182.88"/>
+</segment>
+<segment>

Commit message: Added connector and mosfet for OBS
Parts:
- added LED9: (no value), led:LEDSML0603
- added POWER2: T2I5P, T2I5P:T2I5P
- added R6: 330, resistor:R-US_R0603
- added U1: FQB27P06, CamSensComponents:FQB27P06
Connections:
- new net E_MAG_1: POWER2.4, POWER2.5, R6.2, U1.D2
- new net E_MAG_1_ON: PCB1.GPIO19, U1.G2
- new net N$51: LED9.A, R6.1
- net +5V: now also U1.S2
- net GND: now also LED9.C, POWER2.1, POWER2.2
Other:
- note added: "Electro Mangnet 1"
Changed lines of the file:
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@@
 <?xml version="1.0" encoding="utf-8"?>
 <!DOCTYPE eagle SYSTEM "eagle.dtd">
-<eagle version="8.4.3">
+<eagle version="8.5.0">
 <drawing>
 <settings>
@@
 <part name="C5" library="SparkFun-Passives" deviceset="CAP" device="0603-CAP" value="0.1u"/>
 <part name="C6" library="SparkFun-Passives" deviceset="CAP" device="0603-CAP" value="0.1u"/>
+<part name="U1" library="CamSensComponents" deviceset="FQB27P06" device=""/>
+<part name="R6" library="resistor" deviceset="R-US_" device="R0603" value="330"/>
+<part name="LED9" library="led" deviceset="LED" device="SML0603"/>
+<part name="GND73" library="SparkFun-Aesthetics" deviceset="GND" device=""/>
+<part name="GND78" library="SparkFun-Aesthetics" deviceset="GND" device=""/>
+<part name="POWER2" library="T2I5P" deviceset="T2I5P" device=""/>
 </parts>
 <sheets>
@@
 <plain>
 <text x="20.32" y="-7.62" size="1.778" layer="97">power pins</text>
+<text x="180.34" y="149.86" size="3.81" layer="97">Electro Mangnet 1</text>
 </plain>
 <instances>
@@
 <instance part="C5" gate="G$1" x="114.3" y="177.8" rot="R180"/>
 <instance part="C6" gate="G$1" x="147.32" y="177.8" rot="MR180"/>
+<instance part="U1" gate="G$1" x="190.5" y="132.08"/>
+<instance part="R6" gate="G$1" x="210.82" y="109.22" rot="R90"/>
+<instance part="LED9" gate="G$1" x="210.82" y="99.06"/>
+<instance part="GND73" gate="1" x="210.82" y="86.36"/>
+<instance part="GND78" gate="1" x="172.72" y="109.22" rot="MR0"/>
+<instance part="POWER2" gate="&gt;NAME" x="187.96" y="106.68" rot="R270"/>
 </instances>
 <busses>
@@
 <wire x1="-27.94" y1="83.82" x2="-35.56" y2="83.82" width="0.1524" layer="91"/>
 <label x="-35.56" y="83.82" size="1.778" layer="95"/>
+</segment>
+<segment>
+<pinref part="LED9" gate="G$1" pin="C"/>
+<pinref part="GND73" gate="1" pin="GND"/>
+<wire x1="210.82" y1="88.9" x2="210.82" y2="93.98" width="0.1524" layer="91"/>
+</segment>
+<segment>
+<pinref part="POWER2" gate="&gt;NAME" pin="1"/>
+<pinref part="GND78" gate="1" pin="GND"/>
+<wire x1="182.88" y1="111.76" x2="180.34" y2="111.76" width="0.1524" layer="91"/>
+<pinref part="POWER2" gate="&gt;NAME" pin="2"/>
+<wire x1="180.34" y1="111.76" x2="172.72" y2="111.76" width="0.1524" layer="91"/>
+<wire x1="182.88" y1="109.22" x2="180.34" y2="109.22" width="0.1524" layer="91"/>
+<wire x1="180.34" y1="109.22" x2="180.34" y2="111.76" width="0.1524" layer="91"/>
+<junction x="180.34" y="111.76"/>
 </segment>
 </net>
@@
 <label x="-35.56" y="76.2" size="1.778" layer="95"/>
 </segment>
+<segment>
+<pinref part="U1" gate="G$1" pin="S2"/>
+<wire x1="203.2" y1="137.16" x2="203.2" y2="144.78" width="0.1524" layer="91"/>
+</segment>
 </net>
 <net name="3.3V" class="0">
@@
 </segment>
 </net>
+<net name="N$51" class="0">
+<segment>
+<pinref part="R6" gate="G$1" pin="1"/>
+<pinref part="LED9" gate="G$1" pin="A"/>
+<wire x1="210.82" y1="101.6" x2="210.82" y2="104.14" width="0.1524" layer="91"/>
+</segment>
+</net>
+<net name="E_MAG_1" class="0">
+<segment>
+<pinref part="U1" gate="G$1" pin="D2"/>
+<wire x1="203.2" y1="119.38" x2="203.2" y2="116.84" width="0.1524" layer="91"/>
+<label x="195.58" y="106.68" size="1.778" layer="95"/>
+<pinref part="R6" gate="G$1" pin="2"/>
+<wire x1="210.82" y1="114.3" x2="210.82" y2="116.84" width="0.1524" layer="91"/>
+<wire x1="210.82" y1="116.84" x2="203.2" y2="116.84" width="0.1524" layer="91"/>
+<junction x="203.2" y="116.84"/>
+<pinref part="POWER2" gate="&gt;NAME" pin="4"/>
+<wire x1="182.88" y1="104.14" x2="180.34" y2="104.14" width="0.1524" layer="91"/>
+<wire x1="180.34" y1="104.14" x2="180.34" y2="101.6" width="0.1524" layer="91"/>
+<pinref part="POWER2" gate="&gt;NAME" pin="5"/>
+<wire x1="180.34" y1="101.6" x2="182.88" y2="101.6" width="0.1524" layer="91"/>
+<wire x1="180.34" y1="101.6" x2="180.34" y2="96.52" width="0.1524" layer="91"/>
+<wire x1="180.34" y1="96.52" x2="203.2" y2="96.52" width="0.1524" layer="91"/>
+<junction x="180.34" y="101.6"/>
+<wire x1="203.2" y1="96.52" x2="203.2" y2="116.84" width="0.1524" layer="91"/>
+</segment>
+</net>
+<net name="E_MAG_1_ON" class="0">
+<segment>
+<pinref part="U1" gate="G$1" pin="G2"/>
+<wire x1="190.5" y1="132.08" x2="175.26" y2="132.08" width="0.1524" layer="91"/>
+<label x="175.26" y="132.08" size="1.778" layer="95"/>
+</segment>
+<segment>
+<pinref part="PCB1" gate="G$1" pin="GPIO19"/>
+<wire x1="-208.28" y1="129.54" x2="-200.66" y2="129.54" width="0.1524" layer="91"/>
+</segment>
+</net>
