File: xx_backplane_shield_xi.sch (EAGLE design)
At the start: 31 parts, among them U1 FQB27P06

Commit message: Added servo motor connection
Parts:
- added SV1: (no value), con-lstb:MA03-1
Connections:
- new net SERVO_PWM: PCB1.GPIO13, SV1.1
- net +5V: now also SV1.2
- net GND: now also SV1.3
Changed lines of the file:
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@@
 <?xml version="1.0" encoding="utf-8"?>
 <!DOCTYPE eagle SYSTEM "eagle.dtd">
-<eagle version="8.4.1">
+<eagle version="8.5.2">
 <drawing>
 <settings>
@@
 <part name="GND78" library="SparkFun-Aesthetics" deviceset="GND" device=""/>
 <part name="POWER2" library="T2I5P" deviceset="T2I5P" device=""/>
+<part name="SV1" library="con-lstb" library_urn="urn:adsk.eagle:library:162" deviceset="MA03-1" device="" package3d_urn="urn:adsk.eagle:package:8339/1"/>
 </parts>
 <sheets>
@@
 <instance part="GND78" gate="1" x="172.72" y="109.22" rot="MR0"/>
 <instance part="POWER2" gate="&gt;NAME" x="187.96" y="106.68" rot="R270"/>
+<instance part="SV1" gate="G$1" x="-109.22" y="180.34"/>
 </instances>
 <busses>
@@
 <wire x1="180.34" y1="109.22" x2="180.34" y2="111.76" width="0.1524" layer="91"/>
 <junction x="180.34" y="111.76"/>
+</segment>
+<segment>
+<pinref part="SV1" gate="G$1" pin="3"/>
+<wire x1="-101.6" y1="182.88" x2="-88.9" y2="182.88" width="0.1524" layer="91"/>
+<label x="-96.52" y="182.88" size="1.778" layer="95"/>
 </segment>
 </net>
@@
 <wire x1="203.2" y1="137.16" x2="203.2" y2="144.78" width="0.1524" layer="91"/>
 </segment>
+<segment>
+<pinref part="SV1" gate="G$1" pin="2"/>
+<wire x1="-101.6" y1="180.34" x2="-88.9" y2="180.34" width="0.1524" layer="91"/>
+<label x="-96.52" y="180.34" size="1.778" layer="95"/>
+</segment>
 </net>
 <net name="3.3V" class="0">
@@
 </segment>
 </net>
+<net name="SERVO_PWM" class="0">
+<segment>
+<pinref part="PCB1" gate="G$1" pin="GPIO13"/>
+<wire x1="-208.28" y1="124.46" x2="-193.04" y2="124.46" width="0.1524" layer="91"/>
+<label x="-203.2" y="124.46" size="1.778" layer="95"/>
+</segment>
+<segment>
+<pinref part="SV1" gate="G$1" pin="1"/>
+<wire x1="-101.6" y1="177.8" x2="-88.9" y2="177.8" width="0.1524" layer="91"/>
+<label x="-96.52" y="177.8" size="1.778" layer="95"/>
+</segment>
+</net>
